Commit message: Match the model to the robot as built; remove unused files
Model changes (from measurements and photos of the real robot):
- Upper metal deck on brass pillars with the Jetson under it; deck top
  0.175 m above ground, LiDAR and front OAK-D Lite moved up with it
- Printed adapter plate bolted flat on the deck, triangle to the rear,
  so the SO-101 reaches forward over the LiDAR
- Wrist camera: v2 fixed bracket with the Waveshare 160 deg USB camera
- New tests/export_views.py: merged STL (m and mm), GLB, six renders
- reference_photos/ with the photos the model was matched to

Cleanup:
- Remove the unused v3 OAK tilt-mount meshes and code path
- Remove unused upstream SO-101 MJCF and joint-property copies
- Remove the MuJoCo crash log, .DS_Store files and old test renders;
  add a .gitignore for them

Validated: URDF parses with every mesh resolved, MuJoCo holds the arm
and drives the rover stably for 3 s, exported MJCF reloads.

Co-Authored-By: Claude Opus 5.5 <noreply@anthropic.com>

File: mujoco/so101_rover_sim.urdf (robot description, URDF)
Before this commit: robot so101_rover, 22 links, 21 joints
Links:
- removed link wrist_cam_cradle_link
- removed link wrist_cam_mount_base_link
- added link wrist_cam_bracket_link, mass 0.031; collision box size=0.06 0.03 0.03; visual mesh filename=../meshes/mount/wrist_cam_bracket_v2.stl scale=0.001 0.001 0.001
- added link wrist_camera_link, mass 0.015; visual mesh filename=../meshes/rover/usb_camera.stl
- link arm_mount_plate_link: geometry collision box size=0.102 0.128 0.01; visual mesh filename=../meshes/mount/rover_adapter_plate.stl scale=0.001 0.001 0.001
- link base_link: geometry collision box size=0.205 0.19 0.003; collision box size=0.245 0.23 0.085
Joints:
- removed joint wrist_cam_mount_base_joint
- removed joint wrist_cam_tilt_joint
- added joint wrist_cam_bracket_joint: type fixed, parent arm_gripper_link, child wrist_cam_bracket_link, origin xyz=0 -0.000218 0.00095 rpy=3.14159 0 0
- added joint wrist_camera_joint: type fixed, parent wrist_cam_bracket_link, child wrist_camera_link, origin xyz=0 0 0 rpy=0 0 0
- joint 3d_camera_link_joint: origin xyz=0.06531 0 0.021953 rpy=0 0 0 -> xyz=0.06531 0 0.077 rpy=0 0 0
- joint arm_mount_joint: origin xyz=0.00379955 0 0.0584 rpy=0 0 3.14159 -> xyz=-0.0540207 0 0.1074 rpy=0 0 0
- joint arm_mount_plate_joint: origin xyz=0.0249996 0 0.046 rpy=0 0 0 -> xyz=-0.0752207 0 0.095 rpy=0 0 0
- joint base_lidar_link_joint: origin xyz=0.0398145505519817 0 0.04 rpy=0 0 1.5708 -> xyz=0.0398146 0 0.095 rpy=0 0 1.5708
- joint wrist_camera_optical_joint: origin xyz=0 0.0760144 -0.0210803 rpy=-2.48709 0 -3.14159 -> xyz=0.035 -0.06 0.015 rpy=-1.04206 2.22045e-16 0.677782; parent wrist_cam_cradle_link -> wrist_camera_link

File: urdf/so101_rover.urdf (robot description, URDF)
Before this commit: robot so101_rover, 22 links, 21 joints
Links:
- removed link wrist_cam_cradle_link
- removed link wrist_cam_mount_base_link
- added link wrist_cam_bracket_link, mass 0.031; collision box size=0.06 0.03 0.03; visual mesh filename=package://so101_rover_description/meshes/mount/wrist_cam_br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 scale=0.001 0.001 0.001
- added link wrist_camera_link, mass 0.015; visual mesh filename=package://so101_rover_description/meshes/rover/usb_camera.s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
- link arm_mount_plate_link: geometry collision box size=0.102 0.128 0.01; visual mesh filename=package://so101_rover_description/meshes/mount/rover_adapte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 scale=0.001 0.001 0.001
- link base_link: geometry collision box size=0.205 0.19 0.003; collision box size=0.245 0.23 0.085
Joints:
- removed joint wrist_cam_mount_base_joint
- removed joint wrist_cam_tilt_joint
- added joint wrist_cam_bracket_joint: type fixed, parent arm_gripper_link, child wrist_cam_bracket_link, origin xyz=0 -0.000218 0.00095 rpy=3.14159 0 0
- added joint wrist_camera_joint: type fixed, parent wrist_cam_bracket_link, child wrist_camera_link, origin xyz=0 0 0 rpy=0 0 0
- joint 3d_camera_link_joint: origin xyz=0.06531 0 0.021953 rpy=0 0 0 -> xyz=0.06531 0 0.077 rpy=0 0 0
- joint arm_mount_joint: origin xyz=0.00379955 0 0.0584 rpy=0 0 3.14159 -> xyz=-0.0540207 0 0.1074 rpy=0 0 0
- joint arm_mount_plate_joint: origin xyz=0.0249996 0 0.046 rpy=0 0 0 -> xyz=-0.0752207 0 0.095 rpy=0 0 0
- joint base_lidar_link_joint: origin xyz=0.0398145505519817 0 0.04 rpy=0 0 1.5708 -> xyz=0.0398146 0 0.095 rpy=0 0 1.5708
- joint wrist_camera_optical_joint: origin xyz=0 0.0760144 -0.0210803 rpy=-2.48709 0 -3.14159 -> xyz=0.035 -0.06 0.015 rpy=-1.04206 2.22045e-16 0.677782; parent wrist_cam_cradle_link -> wrist_camera_link

Commit message: Fix model against the photo review; add sim cameras and sensors
From an independent review of the renders against reference_photos/:
- Lower body: cut the Waveshare mesh at its real flat top (0.093 m); its
  2.8 cm top cover is not on the Jetson kit
- Upper deck: 160 mm folded tray with side flanges, ending at the plate's
  rear edge; standoffs under the Jetson
- Arm moved 1 cm rearward (LiDAR to yaw axis 65 mm)
- Wrist USB camera placed where it is tied (rod / U-frame corner)
- Render names were rotated 180 deg; side photos renamed side_right

Simulation:
- New scripts/build_mjcf.py: MJCF with front_camera and wrist_camera,
  gripper_frame site, actuator ranges from joint limits
- Gazebo camera and LiDAR sensors in the URDF
- Passive middle wheels (mass taken out of the body, total 4.46 kg);
  wheel axles exactly 0.040 m up; wheel joint limits
- Removed zero-inertia gripper frame body and schema-invalid leftovers
- tests/check_model.py is now read-only and saves camera images

Co-Authored-By: Claude Opus 5.5 <noreply@anthropic.com>

File: mujoco/so101_rover_sim.urdf (robot description, URDF)
Before this commit: robot so101_rover, 22 links, 21 joints
Links:
- added link left_mid_wheel_link, mass 0.207086; collision cylinder length=0.0426 radius=0.04
- added link right_mid_wheel_link, mass 0.207086; collision cylinder length=0.0426 radius=0.04
- link arm_gripper_frame_link: mass 1e-9 -> None
- link base_link: mass 2.78375064359473 -> 2.36958; geometry collision box size=0.183 0.16 0.003; collision box size=0.245 0.23 0.0565
- link wrist_cam_bracket_link: mass 0.031 -> 0.016; geometry collision box size=0.04 0.075 0.02; visual mesh filename=../meshes/mount/wrist_cam_bracket_v2.stl scale=0.001 0.001 0.001
- link wrist_camera_link: mass 0.015 -> 0.012
Joints:
- added joint left_mid_wheel_link_joint: type continuous, parent base_link, child left_mid_wheel_link, origin xyz=0 0.08726 -0.041212 rpy=1.5708 0 0, axis 0 0 -1, limit effort=0 velocity=32
- added joint right_mid_wheel_link_joint: type continuous, parent base_link, child right_mid_wheel_link, origin xyz=0 -0.08726 -0.041212 rpy=1.5708 0 0, axis 0 0 -1, limit effort=0 velocity=32
- joint 3d_camera_link_joint: axis 0 0 0 -> (none); origin xyz=0.06531 0 0.077 rpy=0 0 0 -> xyz=0.06531 0 0.075788 rpy=0 0 0
- joint arm_mount_joint: origin xyz=-0.0540207 0 0.1074 rpy=0 0 0 -> xyz=-0.0640207 0 0.106188 rpy=0 0 0
- joint arm_mount_plate_joint: origin xyz=-0.0752207 0 0.095 rpy=0 0 0 -> xyz=-0.0852207 0 0.093788 rpy=0 0 0
- joint base_joint: origin xyz=0.000460087791654118 6.50856019576702E-10 0.08 rpy=0 0 0 -> xyz=0.000460088 6.50856e-10 0.081212 rpy=0 0 0
- joint base_lidar_link_joint: axis 0 0 0 -> (none); origin xyz=0.0398146 0 0.095 rpy=0 0 1.5708 -> xyz=0.0398146 0 0.093788 rpy=0 0 1.5708
- joint gripper_frame_joint: axis 0 0 0 -> (none)
- joint left_down_wheel_link_joint: limit (none) -> effort=2.0 velocity=32
- joint left_up_wheel_link_joint: limit (none) -> effort=2.0 velocity=32
- joint right_down_wheel_link_joint: limit (none) -> effort=2.0 velocity=32
- joint right_up_wheel_link_joint: limit (none) -> effort=2.0 velocity=32
- joint wrist_camera_joint: origin xyz=0 0 0 rpy=0 0 0 -> xyz=0.02 -0.09 0.008 rpy=3.14159 -0.496584 1.92518
- joint wrist_camera_optical_joint: origin xyz=0.035 -0.06 0.015 rpy=-1.04206 2.22045e-16 0.677782 -> xyz=0 0 0 rpy=-1.5708 0 -1.5708

File: urdf/so101_rover.urdf (robot description, URDF)
Before this commit: robot so101_rover, 22 links, 21 joints
Links:
- added link left_mid_wheel_link, mass 0.207086; collision cylinder length=0.0426 radius=0.04
- added link right_mid_wheel_link, mass 0.207086; collision cylinder length=0.0426 radius=0.04
- link arm_gripper_frame_link: mass 1e-9 -> None
- link base_link: mass 2.78375064359473 -> 2.36958; geometry collision box size=0.183 0.16 0.003; collision box size=0.245 0.23 0.0565
- link wrist_cam_bracket_link: mass 0.031 -> 0.016; geometry collision box size=0.04 0.075 0.02; visual mesh filename=package://so101_rover_description/meshes/mount/wrist_cam_br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 scale=0.001 0.001 0.001
- link wrist_camera_link: mass 0.015 -> 0.012
Joints:
- added joint left_mid_wheel_link_joint: type continuous, parent base_link, child left_mid_wheel_link, origin xyz=0 0.08726 -0.041212 rpy=1.5708 0 0, axis 0 0 -1, limit effort=0 velocity=32
- added joint right_mid_wheel_link_joint: type continuous, parent base_link, child right_mid_wheel_link, origin xyz=0 -0.08726 -0.041212 rpy=1.5708 0 0, axis 0 0 -1, limit effort=0 velocity=32
- joint 3d_camera_link_joint: axis 0 0 0 -> (none); origin xyz=0.06531 0 0.077 rpy=0 0 0 -> xyz=0.06531 0 0.075788 rpy=0 0 0
- joint arm_mount_joint: origin xyz=-0.0540207 0 0.1074 rpy=0 0 0 -> xyz=-0.0640207 0 0.106188 rpy=0 0 0
- joint arm_mount_plate_joint: origin xyz=-0.0752207 0 0.095 rpy=0 0 0 -> xyz=-0.0852207 0 0.093788 rpy=0 0 0
- joint base_joint: origin xyz=0.000460087791654118 6.50856019576702E-10 0.08 rpy=0 0 0 -> xyz=0.000460088 6.50856e-10 0.081212 rpy=0 0 0
- joint base_lidar_link_joint: axis 0 0 0 -> (none); origin xyz=0.0398146 0 0.095 rpy=0 0 1.5708 -> xyz=0.0398146 0 0.093788 rpy=0 0 1.5708
- joint gripper_frame_joint: axis 0 0 0 -> (none)
- joint left_down_wheel_link_joint: limit (none) -> effort=2.0 velocity=32
- joint left_up_wheel_link_joint: limit (none) -> effort=2.0 velocity=32
- joint right_down_wheel_link_joint: limit (none) -> effort=2.0 velocity=32
- joint right_up_wheel_link_joint: limit (none) -> effort=2.0 velocity=32
- joint wrist_camera_joint: origin xyz=0 0 0 rpy=0 0 0 -> xyz=0.02 -0.09 0.008 rpy=3.14159 -0.496584 1.92518
- joint wrist_camera_optical_joint: origin xyz=0.035 -0.06 0.015 rpy=-1.04206 2.22045e-16 0.677782 -> xyz=0 0 0 rpy=-1.5708 0 -1.5708

Commit message: Second review fixes: camera views, deck shape, Jetson stack, build options
- MuJoCo: collision geometry moved to group 3 so it no longer blocks the
  wrist camera (jaws now fill 12.5% of its image); gradient sky and floor
- Deck: 125 mm flat top with sloped walls, rear edge 27 mm inside the plate
  as in the side photo; Jetson board, pillars and spacers at photo heights
- Wheel velocity servos now track the command (kv 1, 2 Nm limit)
- check_model reads urdf/build_params.json, so every documented build
  option passes; new check that the jaws are visible in the wrist camera
- --arm-facing rear refused below 0.09 m LiDAR clearance; battery moved
  to the lower body behind the Jetson (no room on the deck top)
- front_3q render from the same side as the photo; export no longer
  half-writes on --wrist-mount none
- Gazebo OAK camera at 4:3 (69 x 54 deg); package.xml launch deps and
  Waveshare licence note

Co-Authored-By: Claude Opus 5.5 <noreply@anthropic.com>

File: mujoco/so101_rover_sim.urdf (robot description, URDF)
Before this commit: robot so101_rover, 24 links, 23 joints
Links:
- link base_link: geometry collision box size=0.156 0.125 0.003; collision box size=0.245 0.23 0.0565

File: urdf/so101_rover.urdf (robot description, URDF)
Before this commit: robot so101_rover, 24 links, 23 joints
Links:
- link base_link: geometry collision box size=0.156 0.125 0.003; collision box size=0.245 0.23 0.0565

Commit message: Wrist camera mount for the 25x24 mm Pi-board camera; model it
- scripts/make_wrist_mount.py: TheRobotStudio's official SO-101 wrist
  camera mount with the camera plate redrawn for the Waveshare 160 deg
  camera board: 13.5 x 17 mm lens window on the same optical axis, four
  slotted M2 holes covering 20-21 x 12.5-13.5 mm patterns
- meshes/mount/wrist_cam_mount_pi_board.stl and a print-oriented copy in
  export/print/ (least-overhang orientation, 11 cm3)
- build_urdf.py: --wrist-mount pi (new default) places the mount and
  camera at the official wrist-camera pose; lens direction verified
  (gripper tip 11 deg off axis, jaws fill 27% of the simulated image)
- README: mount, print settings, fasteners

Co-Authored-By: Claude Fable 5.1 <noreply@anthropic.com>

File: mujoco/so101_rover_sim.urdf (robot description, URDF)
Before this commit: robot so101_rover, 24 links, 23 joints
Links:
- removed link wrist_cam_bracket_link
- added link wrist_cam_mount_link, mass 0.014; collision mesh filename=../meshes/mount/wrist_cam_mount_pi_board.stl scale=0.001 0.001 0.001; visual mesh filename=../meshes/mount/wrist_cam_mount_pi_board.stl scale=0.001 0.001 0.001
Joints:
- removed joint wrist_cam_bracket_joint
- added joint wrist_cam_mount_joint: type fixed, parent arm_gripper_link, child wrist_cam_mount_link, origin xyz=-0.015 0.024 -0.0315 rpy=-1.5708 -0.0008 -1.5708
- joint wrist_camera_joint: origin xyz=0.02 -0.09 0.008 rpy=3.14159 -0.496584 1.92518 -> xyz=-0.04941 -0.03813 0.0175 rpy=3.14159 3.67321e-06 1.13399; parent wrist_cam_bracket_link -> wrist_cam_mount_link

File: urdf/so101_rover.urdf (robot description, URDF)
Before this commit: robot so101_rover, 24 links, 23 joints
Links:
- removed link wrist_cam_bracket_link
- added link wrist_cam_mount_link, mass 0.014; collision mesh filename=package://so101_rover_description/meshes/mount/wrist_cam_mo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 scale=0.001 0.001 0.001; visual mesh filename=package://so101_rover_description/meshes/mount/wrist_cam_mo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 scale=0.001 0.001 0.001
Joints:
- removed joint wrist_cam_bracket_joint
- added joint wrist_cam_mount_joint: type fixed, parent arm_gripper_link, child wrist_cam_mount_link, origin xyz=-0.015 0.024 -0.0315 rpy=-1.5708 -0.0008 -1.5708
- joint wrist_camera_joint: origin xyz=0.02 -0.09 0.008 rpy=3.14159 -0.496584 1.92518 -> xyz=-0.04941 -0.03813 0.0175 rpy=3.14159 3.67321e-06 1.13399; parent wrist_cam_bracket_link -> wrist_cam_mount_link

Commit message: Wrist mount variants: sideways offset and auto-aim, with a simulated comparison
- make_wrist_mount.py: --offset widens the plate toward the arm bar so the
  camera sits further from the gripper body; --tilt auto yaws it to centre
  the fingertip; variants registered in meshes/mount/wrist_mounts.json
- build_urdf.py --wrist-variant picks one; camera pose follows the variant
- tests/compare_wrist_mounts.py renders each variant's wrist camera and
  reports body / jaw / floor shares, fingertip position and jaw clearance
- three variants shipped with print files: default (24% body), side20
  (17%), side30_ext10 (15%); none touches the moving jaw

Co-Authored-By: Claude Fable 5.1 <noreply@anthropic.com>

File: mujoco/so101_rover_sim.urdf (robot description, URDF)
Before this commit: robot so101_rover, 24 links, 23 joints
Links:
- link wrist_cam_mount_link: mass 0.014 -> 0.01482

File: urdf/so101_rover.urdf (robot description, URDF)
Before this commit: robot so101_rover, 24 links, 23 joints
Links:
- link wrist_cam_mount_link: mass 0.014 -> 0.01482
